File: kicad/test/test/_saved_test.sch (KiCad schematic (older format))
At the start: 2 parts, among them U1 LSHM, U2 LSHM

Commit message: added feedthrough pcb files
Parts:
- U1, U2: symbol test:LSHM -> _saved_test-rescue:LSHM-test
Changed lines of the file:
@@
 EESchema Schematic File Version 4
-EELAYER 29 0
+LIBS:_saved_test-cache
+EELAYER 26 0
 EELAYER END
 $Descr A4 11693 8268
@@
 $EndDescr
 $Comp
-L test:LSHM U2
+L _saved_test-rescue:LSHM-test U2
 U 1 1 5CA5CA20
 P 5450 3600
@@
 $EndComp
 $Comp
-L test:LSHM U1
+L _saved_test-rescue:LSHM-test U1
 U 1 1 5C92FA02
 P 4850 4250
