File: KiCAD/Station04/Station04.kicad_pcb (KiCad board)
At the start: 4 copper layers, 129.7 x 56.5 mm, 11 parts, among them U1 LSHM-110-02.5-L-DV-A-S-TR, U10 CON-SMA-EDGE, U11 CON-SMA-EDGE, U2 CON-SMA-EDGE, U3 CON-SMA-EDGE, U4 CON-SMA-EDGE, U5 CON-SMA-EDGE, U6 CON-SMA-EDGE, U7 CON-SMA-EDGE, U8 CON-SMA-EDGE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

Commit message: finished station04 and station05
Parts:
- U1: footprint breakout:LSHM-110-02.5-L-DV-A-S-TR -> Station04:LSHM-110-02.5-L-DV-A-S-TR
- U10, U11, U2, U3, U4, U5, U6, U7, U8, U9: footprint breakout:CON-SMA-EDGE -> Station04:CON-SMA-EDGE
Other:
- board text added: "1"
- board text added: "10"
- board text added: "2"
- board text added: "3"
- board text added: "4"
- board text added: "5"
- board text added: "6"
- board text added: "7"
- board text added: "8"
- board text added: "9"
- board text added: "Dylan Oh"
- board text added: "June 2019"
- board text added: "Station04"
