File: KiCAD/Station04/Station04.sch (KiCad schematic (older format))
At the start: 11 parts, among them U1 LSHM-110-02.5-L-DV-A-S-TR, U10 CON-SMA-EDGE, U11 CON-SMA-EDGE, U2 CON-SMA-EDGE, U3 CON-SMA-EDGE, U4 CON-SMA-EDGE, U5 CON-SMA-EDGE, U6 CON-SMA-EDGE, U7 CON-SMA-EDGE, U8 CON-SMA-EDGE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

Commit message: finished station04 and station05
Parts:
- U1: footprint breakout:LSHM-110-02.5-L-DV-A-S-TR -> Station04:LSHM-110-02.5-L-DV-A-S-TR; symbol breakout:LSHM-110-02.5-L-DV-A-S-TR -> Station04-rescue:LSHM-110-02.5-L-DV-A-S-TR-breakout
- U10, U11, U2, U3, U4, U5, U6, U7, U8, U9: footprint breakout:CON-SMA-EDGE -> Station04:CON-SMA-EDGE; symbol breakout:CON-SMA-EDGE -> Station04-rescue:CON-SMA-EDGE-breakout
Changed lines of the file:
@@
 EESchema Schematic File Version 4
-LIBS:breakout-cache
-EELAYER 29 0
+LIBS:Station04-cache
+EELAYER 26 0
 EELAYER END
 $Descr A4 11693 8268
@@
 	3450 4800 3450 4600
 $Comp
-L breakout:LSHM-110-02.5-L-DV-A-S-TR U1
+L Station04-rescue:LSHM-110-02.5-L-DV-A-S-TR-breakout U1
 U 1 1 5D080D78
 P 4850 4100
 F 0 "U1" H 4850 4815 50  0000 C CNN
 F 1 "LSHM-110-02.5-L-DV-A-S-TR" H 4850 4724 50  0000 C CNN
-F 2 "breakout:LSHM-110-02.5-L-DV-A-S-TR" H 4850 4800 50  0001 C CNN
+F 2 "Station04:LSHM-110-02.5-L-DV-A-S-TR" H 4850 4800 50  0001 C CNN
 F 3 "" H 4850 4800 50  0001 C CNN
 	1    4850 4100
@@
 Connection ~ 5250 5200
 $Comp
-L breakout:CON-SMA-EDGE U2
+L Station04-rescue:CON-SMA-EDGE-breakout U2
 U 1 1 5D0FD785
 P 3800 3400
 F 0 "U2" H 3800 2985 50  0000 C CNN
 F 1 "CON-SMA-EDGE" H 3800 3076 50  0000 C CNN
-F 2 "breakout:CON-SMA-EDGE" H 3800 3450 50  0001 C CNN
+F 2 "Station04:CON-SMA-EDGE" H 3800 3450 50  0001 C CNN
 F 3 "" H 3800 3450 50  0001 C CNN
 	1    3800 3400
@@
 $EndComp
 $Comp
-L breakout:CON-SMA-EDGE U3
+L Station04-rescue:CON-SMA-EDGE-breakout U3
 U 1 1 5D0FEA6C
 P 3800 3600
 F 0 "U3" H 3800 3185 50  0000 C CNN
 F 1 "CON-SMA-EDGE" H 3800 3276 50  0000 C CNN
-F 2 "breakout:CON-SMA-EDGE" H 3800 3650 50  0001 C CNN
+F 2 "Station04:CON-SMA-EDGE" H 3800 3650 50  0001 C CNN
 F 3 "" H 3800 3650 50  0001 C CNN
 	1    3800 3600
@@
 $EndComp
 $Comp
-L breakout:CON-SMA-EDGE U4
+L Station04-rescue:CON-SMA-EDGE-breakout U4
 U 1 1 5D0FEE88
 P 3800 3800
 F 0 "U4" H 3800 3385 50  0000 C CNN
 F 1 "CON-SMA-EDGE" H 3800 3476 50  0000 C CNN
-F 2 "breakout:CON-SMA-EDGE" H 3800 3850 50  0001 C CNN
+F 2 "Station04:CON-SMA-EDGE" H 3800 3850 50  0001 C CNN
 F 3 "" H 3800 3850 50  0001 C CNN
 	1    3800 3800
@@
 $EndComp
 $Comp
-L breakout:CON-SMA-EDGE U5
+L Station04-rescue:CON-SMA-EDGE-breakout U5
 U 1 1 5D0FF08E
 P 3800 4000
 F 0 "U5" H 3800 3585 50  0000 C CNN
 F 1 "CON-SMA-EDGE" H 3800 3676 50  0000 C CNN
-F 2 "breakout:CON-SMA-EDGE" H 3800 4050 50  0001 C CNN
+F 2 "Station04:CON-SMA-EDGE" H 3800 4050 50  0001 C CNN
 F 3 "" H 3800 4050 50  0001 C CNN
 	1    3800 4000
@@
 $EndComp
 $Comp
-L breakout:CON-SMA-EDGE U6
+L Station04-rescue:CON-SMA-EDGE-breakout U6
 U 1 1 5D0FF269
 P 3800 4200
 F 0 "U6" H 3800 3785 50  0000 C CNN
 F 1 "CON-SMA-EDGE" H 3800 3876 50  0000 C CNN
-F 2 "breakout:CON-SMA-EDGE" H 3800 4250 50  0001 C CNN
+F 2 "Station04:CON-SMA-EDGE" H 3800 4250 50  0001 C CNN
 F 3 "" H 3800 4250 50  0001 C CNN
 	1    3800 4200
@@
 $EndComp
 $Comp
-L breakout:CON-SMA-EDGE U7
+L Station04-rescue:CON-SMA-EDGE-breakout U7
 U 1 1 5D0FF4B8
 P 3800 4400
 F 0 "U7" H 3800 3985 50  0000 C CNN
 F 1 "CON-SMA-EDGE" H 3800 4076 50  0000 C CNN
-F 2 "breakout:CON-SMA-EDGE" H 3800 4450 50  0001 C CNN
+F 2 "Station04:CON-SMA-EDGE" H 3800 4450 50  0001 C CNN
 F 3 "" H 3800 4450 50  0001 C CNN
 	1    3800 4400
@@
 $EndComp
 $Comp
-L breakout:CON-SMA-EDGE U8
+L Station04-rescue:CON-SMA-EDGE-breakout U8
 U 1 1 5D0FF703
 P 3800 4600
 F 0 "U8" H 3800 4185 50  0000 C CNN
 F 1 "CON-SMA-EDGE" H 3800 4276 50  0000 C CNN
-F 2 "breakout:CON-SMA-EDGE" H 3800 4650 50  0001 C CNN
+F 2 "Station04:CON-SMA-EDGE" H 3800 4650 50  0001 C CNN
 F 3 "" H 3800 4650 50  0001 C CNN
 	1    3800 4600
@@
 $EndComp
 $Comp
-L breakout:CON-SMA-EDGE U9
+L Station04-rescue:CON-SMA-EDGE-breakout U9
 U 1 1 5D0FF936
 P 3800 4800
 F 0 "U9" H 3800 4385 50  0000 C CNN
 F 1 "CON-SMA-EDGE" H 3800 4476 50  0000 C CNN
-F 2 "breakout:CON-SMA-EDGE" H 3800 4850 50  0001 C CNN
+F 2 "Station04:CON-SMA-EDGE" H 3800 4850 50  0001 C CNN
 F 3 "" H 3800 4850 50  0001 C CNN
 	1    3800 4800
@@
 $EndComp
 $Comp
-L breakout:CON-SMA-EDGE U10
+L Station04-rescue:CON-SMA-EDGE-breakout U10
 U 1 1 5D0FFADE
 P 3800 5000
 F 0 "U10" H 3800 4585 50  0000 C CNN
 F 1 "CON-SMA-EDGE" H 3800 4676 50  0000 C CNN
-F 2 "breakout:CON-SMA-EDGE" H 3800 5050 50  0001 C CNN
+F 2 "Station04:CON-SMA-EDGE" H 3800 5050 50  0001 C CNN
 F 3 "" H 3800 5050 50  0001 C CNN
 	1    3800 5000
@@
 $EndComp
 $Comp
-L breakout:CON-SMA-EDGE U11
+L Station04-rescue:CON-SMA-EDGE-breakout U11
 U 1 1 5D0FFD23
 P 3800 5200
 F 0 "U11" H 3800 4785 50  0000 C CNN
 F 1 "CON-SMA-EDGE" H 3800 4876 50  0000 C CNN
-F 2 "breakout:CON-SMA-EDGE" H 3800 5250 50  0001 C CNN
+F 2 "Station04:CON-SMA-EDGE" H 3800 5250 50  0001 C CNN
 F 3 "" H 3800 5250 50  0001 C CNN
 	1    3800 5200
