File: KiCAD/Station05/Station05.sch (KiCad schematic (older format))
At the start: 11 parts, among them U1 CON-SMA-EDGE, U10 CON-SMA-EDGE, U11 LSHM-110-02.5-L-DV-A-S-TR, U2 CON-SMA-EDGE, U3 CON-SMA-EDGE, U4 CON-SMA-EDGE, U5 CON-SMA-EDGE, U6 CON-SMA-EDGE, U7 CON-SMA-EDGE, U8 CON-SMA-EDGE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

Commit message: finished station04 and station05
Parts:
- U1, U10, U2, U3, U4, U5, U6, U7, U8, U9: value CON-SMA-EDGE -> CONSMA001-SMD-G; footprint StationXX:CONSMA001-SMD-G -> Station05:CONSMA001-SMD-G; symbol StationXX:CON-SMA-EDGE -> Station05:CONSMA001-SMD-G
- U11: footprint StationXX:LSHM-110-02.5-L-DV-A-S-TR -> Station05:LSHM-110-02.5-L-DV-A-S-TR; symbol StationXX:LSHM-110-02.5-L-DV-A-S-TR -> Station05-rescue:LSHM-110-02.5-L-DV-A-S-TR-StationXX
Changed lines of the file:
@@
 EESchema Schematic File Version 4
-EELAYER 29 0
+LIBS:Station05-cache
+EELAYER 26 0
 EELAYER END
 $Descr A4 11693 8268
@@
 $EndDescr
 $Comp
-L StationXX:LSHM-110-02.5-L-DV-A-S-TR U11
+L Station05-rescue:LSHM-110-02.5-L-DV-A-S-TR-StationXX U11
 U 1 1 5D10989A
 P 5800 3800
 F 0 "U11" H 5800 4500 50  0000 C CNN
 F 1 "LSHM-110-02.5-L-DV-A-S-TR" H 5800 4400 50  0000 C CNN
-F 2 "StationXX:LSHM-110-02.5-L-DV-A-S-TR" H 5800 4400 50  0001 C CNN
+F 2 "Station05:LSHM-110-02.5-L-DV-A-S-TR" H 5800 4400 50  0001 C CNN
 F 3 "" H 5800 4400 50  0001 C CNN
 	1    5800 3800
@@
 $EndComp
 $Comp
-L StationXX:CON-SMA-EDGE U1
+L Station05:CONSMA001-SMD-G U1
 U 1 1 5D10A3CC
 P 5100 3550
-F 0 "U1" H 6250 3350 50  0000 C CNN
-F 1 "CON-SMA-EDGE" H 5850 3350 50  0000 C CNN
-F 2 "StationXX:CONSMA001-SMD-G" H 5100 3600 50  0001 C CNN
+F 0 "U1" H 6400 3350 50  0000 C CNN
+F 1 "CONSMA001-SMD-G" H 5900 3350 50  0000 C CNN
+F 2 "Station05:CONSMA001-SMD-G" H 5100 3600 50  0001 C CNN
 F 3 "" H 5100 3600 50  0001 C CNN
 	1    5100 3550
@@
 $EndComp
 $Comp
-L StationXX:CON-SMA-EDGE U2
+L Station05:CONSMA001-SMD-G U2
 U 1 1 5D10AFDA
 P 5100 3650
-F 0 "U2" H 6250 3450 50  0000 C CNN
-F 1 "CON-SMA-EDGE" H 5850 3450 50  0000 C CNN
-F 2 "StationXX:CONSMA001-SMD-G" H 5100 3700 50  0001 C CNN
+F 0 "U2" H 6400 3450 50  0000 C CNN
+F 1 "CONSMA001-SMD-G" H 5900 3450 50  0000 C CNN
+F 2 "Station05:CONSMA001-SMD-G" H 5100 3700 50  0001 C CNN
 F 3 "" H 5100 3700 50  0001 C CNN
 	1    5100 3650
@@
 $EndComp
 $Comp
-L StationXX:CON-SMA-EDGE U3
+L Station05:CONSMA001-SMD-G U3
 U 1 1 5D10B247
 P 5100 3750
-F 0 "U3" H 6250 3550 50  0000 C CNN
-F 1 "CON-SMA-EDGE" H 5850 3550 50  0000 C CNN
-F 2 "StationXX:CONSMA001-SMD-G" H 5100 3800 50  0001 C CNN
+F 0 "U3" H 6400 3550 50  0000 C CNN
+F 1 "CONSMA001-SMD-G" H 5900 3550 50  0000 C CNN
+F 2 "Station05:CONSMA001-SMD-G" H 5100 3800 50  0001 C CNN
 F 3 "" H 5100 3800 50  0001 C CNN
 	1    5100 3750
@@
 $EndComp
 $Comp
-L StationXX:CON-SMA-EDGE U4
+L Station05:CONSMA001-SMD-G U4
 U 1 1 5D10B3B5
 P 5100 3850
-F 0 "U4" H 6250 3650 50  0000 C CNN
-F 1 "CON-SMA-EDGE" H 5850 3650 50  0000 C CNN
-F 2 "StationXX:CONSMA001-SMD-G" H 5100 3900 50  0001 C CNN
+F 0 "U4" H 6400 3650 50  0000 C CNN
+F 1 "CONSMA001-SMD-G" H 5900 3650 50  0000 C CNN
+F 2 "Station05:CONSMA001-SMD-G" H 5100 3900 50  0001 C CNN
 F 3 "" H 5100 3900 50  0001 C CNN
 	1    5100 3850
@@
 $EndComp
 $Comp
-L StationXX:CON-SMA-EDGE U5
+L Station05:CONSMA001-SMD-G U5
 U 1 1 5D10B60A
 P 5100 3950
-F 0 "U5" H 6250 3750 50  0000 C CNN
-F 1 "CON-SMA-EDGE" H 5850 3750 50  0000 C CNN
-F 2 "StationXX:CONSMA001-SMD-G" H 5100 4000 50  0001 C CNN
+F 0 "U5" H 6400 3750 50  0000 C CNN
+F 1 "CONSMA001-SMD-G" H 5900 3750 50  0000 C CNN
+F 2 "Station05:CONSMA001-SMD-G" H 5100 4000 50  0001 C CNN
 F 3 "" H 5100 4000 50  0001 C CNN
 	1    5100 3950
@@
 $EndComp
 $Comp
-L StationXX:CON-SMA-EDGE U6
+L Station05:CONSMA001-SMD-G U6
 U 1 1 5D10B772
 P 5100 4050
-F 0 "U6" H 6250 3850 50  0000 C CNN
-F 1 "CON-SMA-EDGE" H 5850 3850 50  0000 C CNN
-F 2 "StationXX:CONSMA001-SMD-G" H 5100 4100 50  0001 C CNN
+F 0 "U6" H 6400 3850 50  0000 C CNN
+F 1 "CONSMA001-SMD-G" H 5900 3850 50  0000 C CNN
+F 2 "Station05:CONSMA001-SMD-G" H 5100 4100 50  0001 C CNN
 F 3 "" H 5100 4100 50  0001 C CNN
 	1    5100 4050
@@
 $EndComp
 $Comp
-L StationXX:CON-SMA-EDGE U7
+L Station05:CONSMA001-SMD-G U7
 U 1 1 5D10B9A1
 P 5100 4150
-F 0 "U7" H 6250 3950 50  0000 C CNN
-F 1 "CON-SMA-EDGE" H 5850 3950 50  0000 C CNN
-F 2 "StationXX:CONSMA001-SMD-G" H 5100 4200 50  0001 C CNN
+F 0 "U7" H 6400 3950 50  0000 C CNN
+F 1 "CONSMA001-SMD-G" H 5900 3950 50  0000 C CNN
+F 2 "Station05:CONSMA001-SMD-G" H 5100 4200 50  0001 C CNN
 F 3 "" H 5100 4200 50  0001 C CNN
 	1    5100 4150
@@
 $EndComp
 $Comp
-L StationXX:CON-SMA-EDGE U8
+L Station05:CONSMA001-SMD-G U8
 U 1 1 5D10BB18
 P 5100 4250
-F 0 "U8" H 6250 4050 50  0000 C CNN
-F 1 "CON-SMA-EDGE" H 5850 4050 50  0000 C CNN
-F 2 "StationXX:CONSMA001-SMD-G" H 5100 4300 50  0001 C CNN
+F 0 "U8" H 6400 4050 50  0000 C CNN
+F 1 "CONSMA001-SMD-G" H 5900 4050 50  0000 C CNN
+F 2 "Station05:CONSMA001-SMD-G" H 5100 4300 50  0001 C CNN
 F 3 "" H 5100 4300 50  0001 C CNN
 	1    5100 4250
@@
 $EndComp
 $Comp
-L StationXX:CON-SMA-EDGE U9
+L Station05:CONSMA001-SMD-G U9
 U 1 1 5D10BD13
 P 5100 4350
-F 0 "U9" H 6250 4150 50  0000 C CNN
-F 1 "CON-SMA-EDGE" H 5850 4150 50  0000 C CNN
-F 2 "StationXX:CONSMA001-SMD-G" H 5100 4400 50  0001 C CNN
+F 0 "U9" H 6400 4150 50  0000 C CNN
+F 1 "CONSMA001-SMD-G" H 5900 4150 50  0000 C CNN
+F 2 "Station05:CONSMA001-SMD-G" H 5100 4400 50  0001 C CNN
 F 3 "" H 5100 4400 50  0001 C CNN
 	1    5100 4350
@@
 $EndComp
 $Comp
-L StationXX:CON-SMA-EDGE U10
+L Station05:CONSMA001-SMD-G U10
 U 1 1 5D10BEF3
 P 5100 4450
-F 0 "U10" H 6250 4250 50  0000 C CNN
-F 1 "CON-SMA-EDGE" H 5850 4250 50  0000 C CNN
-F 2 "StationXX:CONSMA001-SMD-G" H 5100 4500 50  0001 C CNN
+F 0 "U10" H 6400 4250 50  0000 C CNN
+F 1 "CONSMA001-SMD-G" H 5900 4250 50  0000 C CNN
+F 2 "Station05:CONSMA001-SMD-G" H 5100 4500 50  0001 C CNN
 F 3 "" H 5100 4500 50  0001 C CNN
 	1    5100 4450
