File: kicad/feedthrough_pcb/feedthrough_pcb.sch (KiCad schematic (older format))
At the start: 2 parts, among them U1 LSHM-110-02.5-L-DV-A-S-TR, U2 LSHM-110-02.5-L-DV-A-S-TR

Commit message: updated feedthrough pcb
Connections:
- net at U1.1: no longer U2.1
- net at U1.11: no longer U2.11
- net at U1.13: no longer U2.13
- net at U1.15: no longer U2.15
- net at U1.17: no longer U2.17
- net at U1.19: no longer U2.19
- net at U1.3: no longer U2.3
- net at U1.5: no longer U2.5
- net at U1.7: no longer U2.7
- net at U1.9: no longer U2.9
Changed lines of the file:
@@
 EESchema Schematic File Version 4
+LIBS:feedthrough_pcb-cache
 EELAYER 29 0
 EELAYER END
@@
 Wire Wire Line
 	6000 4450 5900 4450
-Wire Wire Line
-	6600 4450 6650 4450
-Wire Wire Line
-	6650 4450 6650 4400
-Wire Wire Line
-	6650 4400 5250 4400
-Wire Wire Line
-	5250 4400 5250 4450
-Wire Wire Line
-	5250 4450 5300 4450
-Wire Wire Line
-	6600 4350 6650 4350
-Wire Wire Line
-	6650 4350 6650 4300
-Wire Wire Line
-	6650 4300 5250 4300
-Wire Wire Line
-	5250 4300 5250 4350
-Wire Wire Line
-	5250 4350 5300 4350
-Wire Wire Line
-	6600 4250 6650 4250
-Wire Wire Line
-	6650 4250 6650 4200
-Wire Wire Line
-	6650 4200 5250 4200
-Wire Wire Line
-	5250 4200 5250 4250
-Wire Wire Line
-	5250 4250 5300 4250
-Wire Wire Line
-	6600 4150 6650 4150
-Wire Wire Line
-	6650 4150 6650 4100
-Wire Wire Line
-	6650 4100 5250 4100
-Wire Wire Line
-	5250 4100 5250 4150
-Wire Wire Line
-	5250 4150 5300 4150
-Wire Wire Line
-	6600 4050 6650 4050
-Wire Wire Line
-	6650 4050 6650 4000
-Wire Wire Line
-	6650 4000 5250 4000
-Wire Wire Line
-	5250 4000 5250 4050
-Wire Wire Line
-	5250 4050 5300 4050
-Wire Wire Line
-	6600 3950 6650 3950
-Wire Wire Line
-	6650 3950 6650 3900
-Wire Wire Line
-	6650 3900 5250 3900
-Wire Wire Line
-	5250 3900 5250 3950
-Wire Wire Line
-	5250 3950 5300 3950
-Wire Wire Line
-	6650 3850 6650 3800
-Wire Wire Line
-	6650 3800 5250 3800
-Wire Wire Line
-	5250 3800 5250 3850
-Wire Wire Line
-	5250 3850 5300 3850
-Wire Wire Line
-	6650 3850 6600 3850
-Wire Wire Line
-	6600 3750 6650 3750
-Wire Wire Line
-	6650 3750 6650 3700
-Wire Wire Line
-	6650 3700 5250 3700
-Wire Wire Line
-	5250 3700 5250 3750
-Wire Wire Line
-	5250 3750 5300 3750
-Wire Wire Line
-	6600 3650 6650 3650
-Wire Wire Line
-	6650 3650 6650 3600
-Wire Wire Line
-	6650 3600 5250 3600
-Wire Wire Line
-	5250 3600 5250 3650
-Wire Wire Line
-	5250 3650 5300 3650
-Wire Wire Line
-	6600 3550 6650 3550
-Wire Wire Line
-	6650 3550 6650 3500
-Wire Wire Line
-	6650 3500 5250 3500
-Wire Wire Line
-	5250 3500 5250 3550
-Wire Wire Line
-	5250 3550 5300 3550
 $EndSCHEMATC

Commit message: updated feedthrough pcb
Parts:
- added U3, U4: LSHM-110-02.5-L-DV-A-S-TR, feedthrough_pcb:LSHM-110-02.5-L-DV-A-S-TR, symbol feedthrough_pcb:LSHM-110-02.5-L-DV-A-S-TR
Connections:
- net GND: now reaches U1.1
- net GND: now also U1.11, U1.13, U1.15, U1.17, U1.19, U1.3, U1.41 (GND), U1.5, U1.7, U1.9, U2.1, U2.11, U2.13, U2.15, U2.17, U2.19, U2.3, U2.41 (GND), U2.5, U2.7, U2.9, U3.1, U3.11, U3.13, U3.15, U3.17, U3.19, U3.3, U3.41 (GND), U3.5, U3.7, U3.9, U4.1, U4.11, U4.13, U4.15, U4.17, U4.19, U4.3, U4.41 (GND), U4.5, U4.7, U4.9
- new net: U3.10, U4.10
- new net: U3.12, U4.12
- new net: U3.14, U4.14
- new net: U3.16, U4.16
- new net: U3.18, U4.18
- new net: U3.2, U4.2
- new net: U3.20, U4.20
- new net: U3.4, U4.4
- new net: U3.6, U4.6
- new net: U3.8, U4.8

Commit message: added 3d models to feedthrough_pcb
Parts:
- added U10, U11, U12, U5, U6, U7, U8, U9: LSHM-110-02.5-L-DV-A-S-TR, feedthrough_pcb:LSHM-110-02.5-L-DV-A-S-TR, symbol feedthrough_pcb-rescue:LSHM-110-02.5-L-DV-A-S-TR-feedthrough_pcb
- U1, U2, U3, U4: symbol feedthrough_pcb:LSHM-110-02.5-L-DV-A-S-TR -> feedthrough_pcb-rescue:LSHM-110-02.5-L-DV-A-S-TR-feedthrough_pcb
Connections:
- wire segments 112 -> 336
