File: KiCAD/Igloo09/Igloo09.kicad_pcb (KiCad board)
At the start: 2 copper layers, 40 x 40 mm, 4 parts, among them U1 TEST_PAD, U2 LSHM-110-01-L-RH-A-S-TR, U3 TEST_PAD, U4 LSHM-110-01-L-RH-A-S-TR

Commit message: added 3d models to Igloo09
Parts:
- U1, U3: footprint Igloo06:TEST_PAD -> Igloo09:TEST_PAD
- U2, U4: footprint Igloo06:LSHM-110-01-L-RH-A-S-TR -> Igloo09:LSHM-110-01-L-RH-A-S-TR
