File: KiCAD/Igloo09/Igloo09.sch (KiCad schematic (older format))
At the start: 4 parts, among them U1 TEST_PAD, U2 LSHM-110-01-L-RH-A-S-TR, U3 TEST_PAD, U4 LSHM-110-01-L-RH-A-S-TR

Commit message: added 3d models to Igloo09
Parts:
- U1, U3: footprint Igloo06:TEST_PAD -> Igloo09:TEST_PAD; symbol Igloo06:TEST_PAD -> Igloo09:TEST_PAD
- U2, U4: footprint Igloo06:LSHM-110-01-L-RH-A-S-TR -> Igloo09:LSHM-110-01-L-RH-A-S-TR; symbol Igloo06:LSHM-110-01-L-RH-A-S-TR -> Igloo09:LSHM-110-01-L-RH-A-S-TR
Changed lines of the file:
@@
 EESchema Schematic File Version 4
-LIBS:Igloo06-cache
+LIBS:Igloo09-cache
 EELAYER 26 0
 EELAYER END
@@
 $EndDescr
 $Comp
-L Igloo06:LSHM-110-01-L-RH-A-S-TR U2
+L Igloo09:LSHM-110-01-L-RH-A-S-TR U2
 U 1 1 5CC8D6AB
 P 3150 4100
 F 0 "U2" H 3150 4815 50  0000 C CNN
 F 1 "LSHM-110-01-L-RH-A-S-TR" H 3150 4724 50  0000 C CNN
-F 2 "Igloo06:LSHM-110-01-L-RH-A-S-TR" H 3150 4700 50  0001 C CNN
+F 2 "Igloo09:LSHM-110-01-L-RH-A-S-TR" H 3150 4700 50  0001 C CNN
 F 3 "" H 3150 4700 50  0001 C CNN
 	1    3150 4100
@@
 $EndComp
 $Comp
-L Igloo06:LSHM-110-01-L-RH-A-S-TR U4
+L Igloo09:LSHM-110-01-L-RH-A-S-TR U4
 U 1 1 5CC8D6ED
 P 4250 4100
 F 0 "U4" H 4250 4815 50  0000 C CNN
 F 1 "LSHM-110-01-L-RH-A-S-TR" H 4250 4724 50  0000 C CNN
-F 2 "Igloo06:LSHM-110-01-L-RH-A-S-TR" H 4250 4700 50  0001 C CNN
+F 2 "Igloo09:LSHM-110-01-L-RH-A-S-TR" H 4250 4700 50  0001 C CNN
 F 3 "" H 4250 4700 50  0001 C CNN
 	1    4250 4100
@@
 Connection ~ 4250 4850
 $Comp
-L Igloo06:TEST_PAD U1
+L Igloo09:TEST_PAD U1
 U 1 1 5CC9A3E3
 P 2600 4100
 F 0 "U1" H 2656 4775 50  0000 C CNN
 F 1 "TEST_PAD" H 2656 4684 50  0000 C CNN
-F 2 "Igloo06:TEST_PAD" H 2600 4650 50  0001 C CNN
+F 2 "Igloo09:TEST_PAD" H 2600 4650 50  0001 C CNN
 F 3 "" H 2600 4650 50  0001 C CNN
 	1    2600 4100
@@
 $EndComp
 $Comp
-L Igloo06:TEST_PAD U3
+L Igloo09:TEST_PAD U3
 U 1 1 5CC9B4AA
 P 3700 4100
 F 0 "U3" H 3756 4775 50  0000 C CNN
 F 1 "TEST_PAD" H 3756 4684 50  0000 C CNN
-F 2 "Igloo06:TEST_PAD" H 3700 4650 50  0001 C CNN
+F 2 "Igloo09:TEST_PAD" H 3700 4650 50  0001 C CNN
 F 3 "" H 3700 4650 50  0001 C CNN
 	1    3700 4100
