File: KiCAD/Slush01/Slush01.kicad_pcb (KiCad board)
At the start: 2 copper layers, 35 x 67 mm, 72 parts, among them IC1 ADR440ARMZ, IC10 AD8237ARMZ, IC11 AD8276ARMZ, IC12 AD8603AUJZ-R2, IC13 AD8237ARMZ, IC14 LM78L05, IC15 ADS1115, IC2 AD8276ARMZ, IC3 AD8603AUJZ-R2, IC4 AD8237ARMZ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

Commit message: started Slush02
Connections:
- J1 pad 1: Net-(C1-Pad1) -> SDA
- J1 pad 2: GNDA -> GND
- J1 pad 4: GND -> GNDA
- J1 pad 5: SDA -> Net-(C1-Pad1)
- J1 pad 6: GND -> SCL
- J1 pad 9: SCL -> GND
Routing:
- net SDA: track 13.1 -> 0.00 mm, vias 2 -> 0
- net SCL: track 12.6 -> 0.00 mm, vias 2 -> 0
- net Net-(C1-Pad1): track 6.18 -> 16.4 mm
- net GNDA: track 36.6 -> 41.2 mm, vias 16 -> 18
- net GND: vias 6 -> 7
Other:
- net class Default: trace_width 0.25 -> 0.1524
- net class Power added: clearance 0.2, trace_width 0.508, via_dia 0.6, via_drill 0.4
- rule trace_min: 0.2 -> 0.1524
