File: KiCAD/Gateway01/Gateway01.kicad_pcb (KiCad board)
At the start: 2 copper layers, 75 x 75 mm, 14 parts, among them U1 LSHM-110-02.5-L-DV-A-S-TR, U10 LSHM-110-02.5-L-DV-A-S-TR, U11 LSHM-110-02.5-L-DV-A-S-TR, U12 LSHM-110-02.5-L-DV-A-S-TR, U13 LSHM-110-02.5-L-DV-A-S-TR, U14 LSHM-110-02.5-L-DV-A-S-TR, U2 LSHM-110-02.5-L-DV-A-S-TR, U3 LSHM-110-02.5-L-DV-A-S-TR, U4 LSHM-110-02.5-L-DV-A-S-TR, U5 LSHM-110-02.5-L-DV-A-S-TR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

Commit message: exposed vias and fixed thermals on Gateway01
Parts:
- U7, U8: value LSHM -> LSHM-110-02.5-L-DV-A-S-TR
