File: KiCAD/Windchill01/Windchill01.kicad_pcb (KiCad board)
At the start: 2 copper layers, 66.8 x 24.5 mm, 22 parts, among them J1 C112640, J2 C112640, J3 Battery_Holder, Q1 MMBT3904, Q2 MMBT3904, U1 LTC6702, U2 PIN_HEADER_2_3

Commit message: finished Windchill01
Parts:
- removed the Q2 at (120.5, 76.2)
- removed the U2 at (96.3, 73.2)
- added C4: 1u, Capacitor_SMD:C_0402_1005Metric, F.Cu at (100.8, 62.9)
- added D1: LED, LED_SMD:LED_0603_1608Metric, F.Cu at (124.7, 79.6)
- added J4: 95278-101A14LF, Windchill01:95278-101A14LF, F.Cu at (98.6, 73.3)
- added Q1: MMBT3904, Package_TO_SOT_SMD:SOT-23, F.Cu at (127.2, 76.2)
- added R13: 4.02k, Resistor_SMD:R_0402_1005Metric, F.Cu at (93.2, 68.2)
- added R14: 102k, Resistor_SMD:R_0402_1005Metric, F.Cu at (93.2, 70.7)
- added R15: 3.4k, Resistor_SMD:R_0402_1005Metric, F.Cu at (93.2, 73.3)
- added R16: 60.4k, Resistor_SMD:R_0402_1005Metric, F.Cu at (100.8, 64.1)
- added R17: 6.8k, Resistor_SMD:R_0402_1005Metric, F.Cu at (93.2, 75.8)
- added R18: 13.7k, Resistor_SMD:R_0402_1005Metric, F.Cu at (93.2, 78.4)
- added R19: 27.4k, Resistor_SMD:R_0402_1005Metric, F.Cu at (93.2, 80.9)
- added U1: AQY221R6V, Windchill01:AQY221R6V, F.Cu at (124.8, 70.1)
- C1: value 330p -> 10n; footprint Capacitor_SMD:C_0805_2012Metric -> Capacitor_SMD:C_0402_1005Metric
- C2: footprint Capacitor_SMD:C_0805_2012Metric -> Capacitor_SMD:C_0402_1005Metric
- C3: value 1u -> 10n; footprint Capacitor_SMD:C_0805_2012Metric -> Capacitor_SMD:C_0402_1005Metric
- R1: value 1k -> 1.8k; footprint Resistor_SMD:R_0805_2012Metric -> Resistor_SMD:R_0402_1005Metric
- R10: value 100k -> 80.6k; footprint Resistor_SMD:R_0805_2012Metric -> Resistor_SMD:R_0402_1005Metric
- R11: value 17k -> 100k; footprint Resistor_SMD:R_0805_2012Metric -> Resistor_SMD:R_0402_1005Metric
- R12: value 360k -> 332; footprint Resistor_SMD:R_0805_2012Metric -> Resistor_SMD:R_0402_1005Metric
- R2: value 100k -> 1M; footprint Resistor_SMD:R_0805_2012Metric -> Resistor_SMD:R_0402_1005Metric
- R3: value 100k -> 6.2M; footprint Resistor_SMD:R_0805_2012Metric -> Resistor_SMD:R_0402_1005Metric
- R4: value 1M -> 100k; footprint Resistor_SMD:R_0805_2012Metric -> Resistor_SMD:R_0402_1005Metric
- R5: value 620k -> 100; footprint Resistor_SMD:R_0805_2012Metric -> Resistor_SMD:R_0402_1005Metric
- R6: value 100k -> 10k; footprint Resistor_SMD:R_0805_2012Metric -> Resistor_SMD:R_0402_1005Metric
- R7: value 72k -> 499k; footprint Resistor_SMD:R_0805_2012Metric -> Resistor_SMD:R_0402_1005Metric
- R8: value 1k -> 180k; footprint Resistor_SMD:R_0805_2012Metric -> Resistor_SMD:R_0402_1005Metric
- R9: value 10k -> 100k; footprint Resistor_SMD:R_0805_2012Metric -> Resistor_SMD:R_0402_1005Metric
- moved C1 49.1 mm to (133.6, 78.7)
- moved R9 48.4 mm to (138.6, 71.5), turned to 0 degrees
- moved R10 44.4 mm to (134.6, 74.6), turned to 270 degrees
- moved R8 44.3 mm to (133.6, 79.7)
- moved C2 36.5 mm to (133.6, 77.6)
- moved R12 33.6 mm to (93.2, 65.7), turned to 180 degrees
- moved R11 13.8 mm to (135.7, 74.6)
- moved R7 12.1 mm to (132.4, 71.4), turned to 90 degrees
- moved R2 11.0 mm to (131.8, 79.2), turned to 90 degrees
- moved R3 10.3 mm to (138.6, 72.6), turned to 180 degrees
- moved Q2 6.77 mm to (138.0, 75.1)
- moved U2 6.62 mm to (132.1, 74.9)
- moved R5 6.54 mm to (124.2, 74.4), turned to 90 degrees
- moved R4 5.53 mm to (126.9, 73.9), turned to 0 degrees
- moved R6 5.23 mm to (121.8, 76.2), turned to 90 degrees
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- renumbered Q1 to Q2, U1 to U2
Connections:
- C1 pad 1: sig -> VDD
- C2 pad 1: /+INA -> GND
- C2 pad 2: GND -> VDD
- C3 pad 1: GND -> +INB
- C3 pad 2: VDD -> GND
- Q2 pad 1: /Vbe1 -> Net-(Q2-Pad1)
- R1 pad 1: Vdiv -> RELAY+
- R10 pad 1: /100ms -> Net-(Q2-Pad1)
- R11 pad 1: /-INB -> Net-(Q2-Pad1)
- R12 pad 1: -INA -> /1ms
- R12 pad 2: GND -> OUTB
- R2 pad 1: GND -> VDD
- R2 pad 2: Vdiv -> -INB
- R3 pad 1: /Vbe1 -> Vdiv
- R3 pad 2: OUTB -> -INA
- R4 pad 1: VDD -> Net-(Q1-Pad1)
- R4 pad 2: /-INB -> OUTA
- R5 pad 1: Vdiv -> Net-(D1-Pad2)
- R5 pad 2: -INA -> OUTA
- R6 pad 1: /Vbe2 -> +INB
- R6 pad 2: /OUTA -> sig
- R7 pad 1: /Vbe2 -> -INA
- R8 pad 1: /1ms -> Vdiv
- R8 pad 2: OUTB -> VDD
- R9 pad 1: /10ms -> GND
- R9 pad 2: OUTB -> Vdiv
- U2 pad 1: /OUTA -> OUTA
- U2 pad 3: /+INA -> +INA
- U2 pad 5: sig -> +INB
- U2 pad 6: /-INB -> -INB
Routing:
- net sig: track 0.00 -> 72.2 mm, vias 0 -> 2
- net OUTB: track 0.00 -> 52.5 mm, vias 0 -> 4
- net -INB: track 0.00 -> 51.2 mm, vias 0 -> 2
- net +INA: track 0.00 -> 40.9 mm, vias 0 -> 2
- net -INA: track 0.00 -> 23.8 mm, vias 0 -> 1
- net VDD: track 0.00 -> 20.6 mm, vias 0 -> 2
- net OUTA: track 0.00 -> 16.2 mm, vias 0 -> 1
- net +INB: track 0.00 -> 12.6 mm
- net Vdiv: track 0.00 -> 10.9 mm
- net RELAY-: track 0.00 -> 10.8 mm, vias 0 -> 2
- net Net-(D1-Pad2): track 0.00 -> 7.64 mm, vias 0 -> 2
- net Net-(Q2-Pad1): track 0.00 -> 2.46 mm
- net /80mV: track 0.00 -> 2.12 mm
- net /40mV: track 0.00 -> 2.12 mm
- net /20mV: track 0.00 -> 2.12 mm
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- added copper zone on B.Cu, net GND
- added copper zone on F.Cu, net GND
Other:
- board size 66.8 x 24.5 mm -> 66.8 x 24.6 mm
- board text added: "(Gusting when lit)"
- board text added: "1"
- board text added: "10"
- board text added: "100"
- board text added: "20"
- board text added: "40"
- board text added: "80"
- board text added: "Comparator 1 Test Points"
- board text added: "Comparator 2 Test Points"
- board text added: "Cooling SNSPDs down"
- board text added: "Dylan Oh"
- board text added: "Output to RC"
- board text added: "RC Circuit (+IN)"
- board text added: "Restart Delay"
- board text added: "Signal (+IN)"
- board text added: "Switching Voltage"
- board text added: "Tau Threshold V (-IN)"
- board text added: "Threshold V (-IN)"
- board text added: "Threshold Voltage Set"
- board text added: "Windchill01"
- board text added: "[mV]"
- board text added: "[ms]"
- board text added: "since August 2019"
- board text removed: "1 ms"
- board text removed: "10 ms"
- board text removed: "100 ms"
