File: KiCAD/Windchill01/Windchill01.kicad_pcb (KiCad board)
At the start: 2 copper layers, 66.8 x 24.6 mm, 32 parts, among them J1 C112640, J2 C112640, J3 Battery_Holder, J4 95278-101A14LF, Q1 MMBT3904, Q2 MMBT3904, U1 AQY221R6V, U2 LTC6702

Commit message: readded wind graphic
Parts:
- added G1: Wind_Graphic, Windchill01:wind, F.Cu at (131.4, 65.6)

Commit message: finished Windchill01 for real this time
Routing:
- net sig: track 72.2 -> 82.4 mm, vias 2 -> 4
Changed lines of the file:
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@@
     (thickness 1.6)
     (drawings 90)
-    (tracks 174)
+    (tracks 176)
     (zones 0)
     (modules 33)
@@
   (segment (start 119.752 71.495) (end 119.752 74.752) (width 0.25) (layer F.Cu) (net 1))
   (segment (start 121.8 75.72) (end 120.72 75.72) (width 0.25) (layer F.Cu) (net 1) (status 10))
-  (segment (start 144.6 72.397) (end 144.6 73.22) (width 0.25) (layer F.Cu) (net 1) (status 20))
-  (segment (start 123.288 70.752) (end 125.32 68.72) (width 0.25) (layer F.Cu) (net 1))
-  (segment (start 122.588 70.752) (end 123.288 70.752) (width 0.25) (layer F.Cu) (net 1) (status 10))
-  (segment (start 125.32 68.72) (end 127.6315 68.72) (width 0.25) (layer F.Cu) (net 1))
-  (segment (start 127.6315 68.72) (end 128.2615 69.35) (width 0.25) (layer F.Cu) (net 1))
-  (segment (start 128.2615 69.35) (end 141.553 69.35) (width 0.25) (layer F.Cu) (net 1))
-  (segment (start 141.553 69.35) (end 144.6 72.397) (width 0.25) (layer F.Cu) (net 1))
+  (segment (start 144.6 72.54) (end 140.41 68.35) (width 0.25) (layer F.Cu) (net 1))
+  (segment (start 144.6 73.22) (end 144.6 72.54) (width 0.25) (layer F.Cu) (net 1))
+  (via (at 139.86 63.13) (size 0.8) (drill 0.4) (layers F.Cu B.Cu) (net 1))
+  (segment (start 140.41 68.35) (end 140.41 63.68) (width 0.25) (layer F.Cu) (net 1))
+  (segment (start 140.41 63.68) (end 139.86 63.13) (width 0.25) (layer F.Cu) (net 1))
+  (segment (start 139.86 63.13) (end 126.72 63.13) (width 0.25) (layer B.Cu) (net 1))
+  (via (at 120.495 70.752) (size 0.8) (drill 0.4) (layers F.Cu B.Cu) (net 1))
+  (segment (start 126.72 63.13) (end 120.495 69.355) (width 0.25) (layer B.Cu) (net 1))
+  (segment (start 120.495 69.355) (end 120.495 70.752) (width 0.25) (layer B.Cu) (net 1))
   (via (at 135.7 76.8) (size 0.8) (drill 0.4) (layers F.Cu B.Cu) (net 2))
   (via (at 129.342 73.281) (size 0.8) (drill 0.4) (layers F.Cu B.Cu) (net 2))
