File: KiCAD/Windchill01/Windchill01.sch (KiCad schematic (older format))
At the start: 22 parts, among them J1 C112640, J2 C112640, J3 Battery_Holder, Q1 MMBT3904, Q2 MMBT3904, U1 LTC6702, U2 PIN_HEADER_2_3

Commit message: finished Windchill01
Parts:
- removed R7: 72k, Resistor_SMD:R_0805_2012Metric, symbol Device:R_US
- removed U2: PIN_HEADER_2_3, Windchill01:95278-101A06LF, symbol Windchill01:PIN_HEADER_2_3
- added C1: 10n, Capacitor_SMD:C_0402_1005Metric, symbol Device:C
- added D1: LED, LED_SMD:LED_0603_1608Metric, symbol Device:LED
- added J4: 95278-101A14LF, Windchill01:95278-101A14LF, symbol Windchill01:95278-101A14LF
- added R1: 1.8k, Resistor_SMD:R_0402_1005Metric, symbol Device:R_US
- added R15: 3.4k, Resistor_SMD:R_0402_1005Metric, symbol Device:R_US
- added R16: 60.4k, Resistor_SMD:R_0402_1005Metric, symbol Device:R_US
- added R17: 6.8k, Resistor_SMD:R_0402_1005Metric, symbol Device:R_US
- added R18: 13.7k, Resistor_SMD:R_0402_1005Metric, symbol Device:R_US
- added R19: 27.4k, Resistor_SMD:R_0402_1005Metric, symbol Device:R_US
- added R5: 100, Resistor_SMD:R_0402_1005Metric, symbol Device:R_US
- added R6: 10k, Resistor_SMD:R_0402_1005Metric, symbol Device:R_US
- added U1: AQY221R6V, Windchill01:AQY221R6V, symbol Windchill01:AQY221R6V
- C2: renamed from C3; footprint Capacitor_SMD:C_0805_2012Metric -> Capacitor_SMD:C_0402_1005Metric
- C3: renamed from C1; value 330p -> 10n; footprint Capacitor_SMD:C_0805_2012Metric -> Capacitor_SMD:C_0402_1005Metric
- C4: renamed from C2; footprint Capacitor_SMD:C_0805_2012Metric -> Capacitor_SMD:C_0402_1005Metric
- R10: renamed from R3; value 100k -> 80.6k; footprint Resistor_SMD:R_0805_2012Metric -> Resistor_SMD:R_0402_1005Metric
- R11: value 17k -> 100k; footprint Resistor_SMD:R_0805_2012Metric -> Resistor_SMD:R_0402_1005Metric
- R12: renamed from R8; value 1k -> 332; footprint Resistor_SMD:R_0805_2012Metric -> Resistor_SMD:R_0402_1005Metric
- R13: renamed from R9; value 10k -> 4.02k; footprint Resistor_SMD:R_0805_2012Metric -> Resistor_SMD:R_0402_1005Metric
- R14: renamed from R10; value 100k -> 102k; footprint Resistor_SMD:R_0805_2012Metric -> Resistor_SMD:R_0402_1005Metric
- R2: renamed from R4; footprint Resistor_SMD:R_0805_2012Metric -> Resistor_SMD:R_0402_1005Metric
- R3: renamed from R5; value 620k -> 6.2M; footprint Resistor_SMD:R_0805_2012Metric -> Resistor_SMD:R_0402_1005Metric
- R4: renamed from R6; footprint Resistor_SMD:R_0805_2012Metric -> Resistor_SMD:R_0402_1005Metric
- R7: renamed from R12; value 360k -> 499k; footprint Resistor_SMD:R_0805_2012Metric -> Resistor_SMD:R_0402_1005Metric
- R8: renamed from R1; value 1k -> 180k; footprint Resistor_SMD:R_0805_2012Metric -> Resistor_SMD:R_0402_1005Metric
- R9: renamed from R2; footprint Resistor_SMD:R_0805_2012Metric -> Resistor_SMD:R_0402_1005Metric
- renumbered Q2 to Q1, Q1 to Q2, U1 to U2
Connections:
- net labels added: +INB, 10mV, 20mV, 40mV, 80mV, RELAY+, RELAY-
- net labels removed: Vbe1, Vbe2
- wire segments 73 -> 123
Other:
- moved on the sheet: C2, C3, C4, J1, J2, J3, Q1, Q2, R10, R12, R13, R14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

Commit message: readded wind graphic
Parts:
- added G1: Wind_Graphic, Windchill01:wind, symbol Windchill01:Wind_Graphic
Changed lines of the file:
@@
 EESchema Schematic File Version 4
-LIBS:Windchill01-cache
 EELAYER 30 0
 EELAYER END
@@
 Text GLabel 4850 2500 0    50   Input ~ 0
 RELAY-
+$Comp
+L Windchill01:Wind_Graphic G1
+U 1 1 5D5BAF4A
+P 6450 3250
+F 0 "G1" H 6475 3296 50  0000 L CNN
+F 1 "Wind_Graphic" H 6475 3205 50  0000 L CNN
+F 2 "Windchill01:wind" H 6450 3250 50  0001 C CNN
+F 3 "" H 6450 3250 50  0001 C CNN
+	1    6450 3250
+	1    0    0    -1
+$EndComp
 $EndSCHEMATC
