File: KiCAD/Slush02/_autosave-Slush02.sch (KiCad schematic (older format))
At the start: 12 parts, among them IC1 ADR440ARMZ, IC14 LM78L05, IC15 ADS1115, J1 DB9F, J2 90122-0128

Commit message: started Slush02
Parts:
- C1, C2, C3, C33, C4: footprint Capacitor_SMD:C_0805_2012Metric_Pad1.15x1.40mm_HandSolder -> Capacitor_SMD:C_0402_1005Metric
- IC1: footprint Slush01:MSOP-8 -> Slush02:MSOP-8; symbol Slush01:ADR440ARMZ -> Slush02:ADR440ARMZ
- IC14: footprint Slush01:SOIC-8 -> Slush02:SOIC-8; symbol Slush01:LM78L05 -> Slush02:LM78L05
- IC15: footprint Slush01:VSSOP-10 -> Slush02:VSSOP-10; symbol Slush01:ADS1115 -> Slush02:ADS1115
- J1: footprint Slush01:K202XHT-E9S-N -> Slush02:K202XHT-E9S-N; symbol Slush01:DB9F -> Slush02:DB9F
- J2: footprint Slush01:90122-0128 -> Slush02:90122-0128; symbol Slush01:90122-0128 -> Slush02:90122-0128
- R1, R2: footprint Resistor_SMD:R_0805_2012Metric_Pad1.15x1.40mm_HandSolder -> Resistor_SMD:R_0402_1005Metric
Connections:
- wire segments 132 -> 134
- no-connect marks 1 -> 2
Changed lines of the file:
@@
 EESchema Schematic File Version 4
+LIBS:Slush02-cache
 EELAYER 30 0
 EELAYER END
@@
 F 0 "R1" V 7230 3400 50  0000 C CNN
 F 1 "1050" V 7150 3400 50  0000 C CNN
-F 2 "Resistor_SMD:R_0805_2012Metric_Pad1.15x1.40mm_HandSolder" V 7080 3400 50  0001 C CNN
+F 2 "Resistor_SMD:R_0402_1005Metric" V 7080 3400 50  0001 C CNN
 F 3 "" H 7150 3400 50  0001 C CNN
 F 4 "-" H -2150 -450 50  0001 C CNN "MFR"
@@
 F 0 "R2" V 7230 3750 50  0000 C CNN
 F 1 "1K" V 7150 3750 50  0000 C CNN
-F 2 "Resistor_SMD:R_0805_2012Metric_Pad1.15x1.40mm_HandSolder" V 7080 3750 50  0001 C CNN
+F 2 "Resistor_SMD:R_0402_1005Metric" V 7080 3750 50  0001 C CNN
 F 3 "" H 7150 3750 50  0001 C CNN
 F 4 "-" H -2150 -450 50  0001 C CNN "MFR"
@@
 F 0 "C3" H 5525 3450 50  0000 L CNN
 F 1 "0.1uF" H 5525 3250 50  0000 L TNN
-F 2 "Capacitor_SMD:C_0805_2012Metric_Pad1.15x1.40mm_HandSolder" H 5538 3200 50  0001 C CNN
+F 2 "Capacitor_SMD:C_0402_1005Metric" H 5538 3200 50  0001 C CNN
 F 3 "" H 5500 3350 50  0001 C CNN
 F 4 "-" H -2050 -50 50  0001 C CNN "MFR"
@@
 F 0 "C4" H 7475 3600 50  0000 L CNN
 F 1 "0.1uF" H 7475 3400 50  0000 L TNN
-F 2 "Capacitor_SMD:C_0805_2012Metric_Pad1.15x1.40mm_HandSolder" H 7488 3350 50  0001 C CNN
+F 2 "Capacitor_SMD:C_0402_1005Metric" H 7488 3350 50  0001 C CNN
 F 3 "" H 7450 3500 50  0001 C CNN
 F 4 "-" H -2150 -450 50  0001 C CNN "MFR"
@@
 F 0 "C1" H 3942 1596 50  0000 L CNN
 F 1 "0.33uF" H 3942 1505 50  0000 L CNN
-F 2 "Capacitor_SMD:C_0805_2012Metric_Pad1.15x1.40mm_HandSolder" H 3850 1550 50  0001 C CNN
+F 2 "Capacitor_SMD:C_0402_1005Metric" H 3850 1550 50  0001 C CNN
 F 3 "~" H 3850 1550 50  0001 C CNN
 	1    3850 1550
@@
 F 0 "C2" H 4742 1596 50  0000 L CNN
 F 1 "0.01uF" H 4742 1505 50  0000 L CNN
-F 2 "Capacitor_SMD:C_0805_2012Metric_Pad1.15x1.40mm_HandSolder" H 4650 1550 50  0001 C CNN
+F 2 "Capacitor_SMD:C_0402_1005Metric" H 4650 1550 50  0001 C CNN
 F 3 "~" H 4650 1550 50  0001 C CNN
 	1    4650 1550
@@
 	5850 3350 5850 3550
 $Comp
-L Slush01:ADR440ARMZ IC1
+L Slush02:ADR440ARMZ IC1
 U 1 1 5D42964B
 P 5850 3050
 F 0 "IC1" H 6350 3317 50  0000 C CNN
 F 1 "ADR440ARMZ" H 6350 3226 50  0000 C CNN
-F 2 "Slush01:MSOP-8" H 6350 2500 50  0001 C CNN
+F 2 "Slush02:MSOP-8" H 6350 2500 50  0001 C CNN
 F 3 "http://docs-europe.electrocomponents.com/webdocs/0de0/0900766b80de0ad0.pdf" H 6350 2400 50  0001 C CNN
 F 4 "V-Ref Precision 2.048V 10mA 8-Pin MSOP" H 6350 2300 50  0001 C CNN "Description"
@@
 $EndComp
 $Comp
-L Slush01:DB9F J1
+L Slush02:DB9F J1
 U 1 1 5D42E11B
 P 2900 1850
 F 0 "J1" H 2820 2542 50  0000 C CNN
 F 1 "DB9F" H 2820 2451 50  0000 C CNN
-F 2 "Slush01:K202XHT-E9S-N" H 2900 1850 50  0001 C CNN
+F 2 "Slush02:K202XHT-E9S-N" H 2900 1850 50  0001 C CNN
 F 3 "" H 2900 1850 50  0001 C CNN
 	1    2900 1850
@@
 $EndComp
 $Comp
-L Slush01:90122-0128 J2
+L Slush02:90122-0128 J2
 U 1 1 5D72D6A3
 P 1500 5600
 F 0 "J2" H 1681 7375 50  0000 C CNN
 F 1 "90122-0128" H 1681 7284 50  0000 C CNN
-F 2 "Slush01:90122-0128" H 1650 6000 50  0001 C CNN
+F 2 "Slush02:90122-0128" H 1650 6000 50  0001 C CNN
 F 3 "" H 1650 6000 50  0001 C CNN
 	1    1500 5600
@@
 	3300 1550 3300 1750
 $Comp
-L Slush01:LM78L05 IC14
+L Slush02:LM78L05 IC14
 U 1 1 5D43B63A
 P 4250 1500
 F 0 "IC14" H 4250 1792 50  0000 C CNN
 F 1 "LM78L05" H 4250 1701 50  0000 C CNN
-F 2 "Slush01:SOIC-8" H 4250 1800 50  0001 C CNN
+F 2 "Slush02:SOIC-8" H 4250 1800 50  0001 C CNN
 F 3 "" H 4250 1800 50  0001 C CNN
 	1    4250 1500
@@
 $EndComp
 $Comp
-L Slush01:ADS1115 IC15
+L Slush02:ADS1115 IC15
 U 1 1 5D449C03
 P 5950 4750
 F 0 "IC15" H 5950 5378 50  0000 C CNN
 F 1 "ADS1115" H 5950 5287 50  0000 C CNN
-F 2 "Slush01:VSSOP-10" H 5950 4750 50  0001 C CNN
+F 2 "Slush02:VSSOP-10" H 5950 4750 50  0001 C CNN
 F 3 "" H 5950 4750 50  0001 C CNN
 	1    5950 4750
@@
 	4450 5350 5200 5350
 Wire Wire Line
-	5200 4800 5550 4800
-Wire Wire Line
-	5200 4400 5200 4800
-Wire Wire Line
 	5200 4900 5550 4900
 Wire Wire Line
@@
 Wire Wire Line
 	4450 3450 5400 3450
-Wire Wire Line
-	5400 3450 5400 4700
-Wire Wire Line
-	5400 4700 5550 4700
 Wire Wire Line
 	5950 4300 5950 4100
@@
 F 0 "C33" H 6225 4200 50  0000 L CNN
 F 1 "0.1uF" H 6225 4000 50  0000 L TNN
-F 2 "Capacitor_SMD:C_0805_2012Metric_Pad1.15x1.40mm_HandSolder" H 6238 3950 50  0001 C CNN
+F 2 "Capacitor_SMD:C_0402_1005Metric" H 6238 3950 50  0001 C CNN
 F 3 "" H 6200 4100 50  0001 C CNN
 F 4 "-" H -1350 700 50  0001 C CNN "MFR"
@@
 Wire Wire Line
 	2900 1250 2900 1200
-$Comp
-L power:GND #PWR0152
-U 1 1 5D49CEC6
-P 2900 1200
-F 0 "#PWR0152" H 2900 950 50  0001 C CNN
-F 1 "GND" H 2905 1027 50  0000 C CNN
-F 2 "" H 2900 1200 50  0001 C CNN
-F 3 "" H 2900 1200 50  0001 C CNN
-	1    2900 1200
-	-1   0    0    1
-$EndComp
 Wire Wire Line
 	3200 1750 3300 1750
@@
 Wire Wire Line
 	3300 2050 3300 2550
+NoConn ~ 3200 1850
+Wire Wire Line
+	2900 1200 3300 1200
+Wire Wire Line
+	3300 1200 3300 1550
+Connection ~ 3300 1550
+Wire Wire Line
+	5200 4400 5200 4800
+Wire Wire Line
+	5400 3450 5400 4700
+Wire Wire Line
+	5400 4700 5550 4700
+Wire Wire Line
+	5200 4800 5550 4800
 $EndSCHEMATC
