File: KiCAD/Slush02/channel.sch (KiCad schematic (older format))
At the start: 15 parts, among them IC11 AD8276ARMZ, IC12 AD8603AUJZ-R2, IC13 AD8237ARMZ

Commit message: started Slush02
Parts:
- C26, C27, C28, C29, C30, C31: footprint Capacitor_SMD:C_0805_2012Metric_Pad1.15x1.40mm_HandSolder -> Capacitor_SMD:C_0402_1005Metric
- C32: footprint Capacitor_Tantalum_SMD:CP_EIA-3216-18_Kemet-A_Pad1.58x1.35mm_HandSolder -> Capacitor_Tantalum_SMD:CP_EIA-2012-12_Kemet-R
- IC11: footprint Slush01:MSOP-8 -> Slush02:MSOP-8; symbol Slush01:AD8276ARMZ -> Slush02:AD8276ARMZ
- IC12: footprint Slush01:TSOT-23-5 -> Slush02:TSOT-23-5; symbol Slush01:AD8603AUJZ-R2 -> Slush02:AD8603AUJZ-R2
- IC13: footprint Slush01:MSOP-8 -> Slush02:MSOP-8; symbol Slush01:AD8237ARMZ -> Slush02:AD8237ARMZ
- R19, R20, R21, R22: footprint Resistor_SMD:R_0805_2012Metric_Pad1.15x1.40mm_HandSolder -> Resistor_SMD:R_0402_1005Metric
Changed lines of the file:
@@
 AR Path="/59ED3D94/59ED1256" Ref="R7"  Part="1"
 AR Path="/59ED3DAD/59ED1256" Ref="R11"  Part="1"
-F 0 "R7" V 4130 3250 50  0000 C CNN
+F 0 "R19" V 4130 3250 50  0000 C CNN
 F 1 "100k" V 4050 3250 50  0000 C CNN
-F 2 "Resistor_SMD:R_0805_2012Metric_Pad1.15x1.40mm_HandSolder" V 3980 3250 50  0001 C CNN
+F 2 "Resistor_SMD:R_0402_1005Metric" V 3980 3250 50  0001 C CNN
 F 3 "" H 4050 3250 50  0001 C CNN
 F 4 "Yageo" H 0   0   50  0001 C CNN "MFR"
@@
 AR Path="/59ED3D94/59ED125E" Ref="R10"  Part="1"
 AR Path="/59ED3DAD/59ED125E" Ref="R14"  Part="1"
-F 0 "R10" V 4130 3900 50  0000 C CNN
+F 0 "R22" V 4130 3900 50  0000 C CNN
 F 1 "10k" V 4050 3900 50  0000 C CNN
-F 2 "Resistor_SMD:R_0805_2012Metric_Pad1.15x1.40mm_HandSolder" V 3980 3900 50  0001 C CNN
+F 2 "Resistor_SMD:R_0402_1005Metric" V 3980 3900 50  0001 C CNN
 F 3 "" H 4050 3900 50  0001 C CNN
 F 4 "Yageo" H 0   0   50  0001 C CNN "MFR"
@@
 AR Path="/59ED3D94/59ED1265" Ref="R8"  Part="1"
 AR Path="/59ED3DAD/59ED1265" Ref="R12"  Part="1"
-F 0 "R8" V 4430 3500 50  0000 C CNN
+F 0 "R20" V 4430 3500 50  0000 C CNN
 F 1 "100k" V 4350 3500 50  0000 C CNN
-F 2 "Resistor_SMD:R_0805_2012Metric_Pad1.15x1.40mm_HandSolder" V 4280 3500 50  0001 C CNN
+F 2 "Resistor_SMD:R_0402_1005Metric" V 4280 3500 50  0001 C CNN
 F 3 "" H 4350 3500 50  0001 C CNN
 F 4 "Yageo" H 0   0   50  0001 C CNN "MFR"
@@
 AR Path="/59ED3D94/59ED126C" Ref="R9"  Part="1"
 AR Path="/59ED3DAD/59ED126C" Ref="R13"  Part="1"
-F 0 "R9" V 4430 3700 50  0000 C CNN
+F 0 "R21" V 4430 3700 50  0000 C CNN
 F 1 "100k" V 4350 3700 50  0000 C CNN
-F 2 "Resistor_SMD:R_0805_2012Metric_Pad1.15x1.40mm_HandSolder" V 4280 3700 50  0001 C CNN
+F 2 "Resistor_SMD:R_0402_1005Metric" V 4280 3700 50  0001 C CNN
 F 3 "" H 4350 3700 50  0001 C CNN
 F 4 "Yageo" H 0   0   50  0001 C CNN "MFR"
@@
 AR Path="/59ED3D94/59ED1273" Ref="C9"  Part="1"
 AR Path="/59ED3DAD/59ED1273" Ref="C16"  Part="1"
-F 0 "C9" H 4775 3950 50  0000 L CNN
+F 0 "C30" H 4775 3950 50  0000 L CNN
 F 1 "0.1uF" H 4775 3750 50  0000 L CNN
-F 2 "Capacitor_SMD:C_0805_2012Metric_Pad1.15x1.40mm_HandSolder" H 4788 3700 50  0001 C CNN
+F 2 "Capacitor_SMD:C_0402_1005Metric" H 4788 3700 50  0001 C CNN
 F 3 "" H 4750 3850 50  0001 C CNN
 F 4 "CL21B104KOANNNC" H 0   0   50  0001 C CNN "MPN"
@@
 AR Path="/59ED3D94/59ED127A" Ref="C7"  Part="1"
 AR Path="/59ED3DAD/59ED127A" Ref="C14"  Part="1"
-F 0 "C7" H 4775 3450 50  0000 L CNN
+F 0 "C28" H 4775 3450 50  0000 L CNN
 F 1 "0.1uF" H 4850 3350 50  0000 L CNN
-F 2 "Capacitor_SMD:C_0805_2012Metric_Pad1.15x1.40mm_HandSolder" H 4788 3200 50  0001 C CNN
+F 2 "Capacitor_SMD:C_0402_1005Metric" H 4788 3200 50  0001 C CNN
 F 3 "" H 4750 3350 50  0001 C CNN
 F 4 "GRM31C5C1E104JA01L " H 4750 3350 60  0001 C CNN "Part"
@@
 AR Path="/59ED3D94/59ED1281" Ref="C8"  Part="1"
 AR Path="/59ED3DAD/59ED1281" Ref="C15"  Part="1"
-F 0 "C8" H 5025 3700 50  0000 L CNN
+F 0 "C29" H 5025 3700 50  0000 L CNN
 F 1 "1uF 6.3V X7R 0805" H 5025 3500 50  0000 L CNN
-F 2 "Capacitor_SMD:C_0805_2012Metric_Pad1.15x1.40mm_HandSolder" H 5038 3450 50  0001 C CNN
+F 2 "Capacitor_SMD:C_0402_1005Metric" H 5038 3450 50  0001 C CNN
 F 3 "" H 5000 3600 50  0001 C CNN
 F 4 "CC0805KKX7R8BB105" H 5000 3600 60  0001 C CNN "MPN"
@@
 AR Path="/59ED3D94/59ED1AD1" Ref="C10"  Part="1"
 AR Path="/59ED3DAD/59ED1AD1" Ref="C17"  Part="1"
-F 0 "C10" H 6375 4150 50  0000 L CNN
+F 0 "C31" H 6375 4150 50  0000 L CNN
 F 1 "0.1uF" H 6100 3950 50  0000 L CNN
-F 2 "Capacitor_SMD:C_0805_2012Metric_Pad1.15x1.40mm_HandSolder" H 6388 3900 50  0001 C CNN
+F 2 "Capacitor_SMD:C_0402_1005Metric" H 6388 3900 50  0001 C CNN
 F 3 "" H 6350 4050 50  0001 C CNN
 F 4 "Samsung" H 0   0   50  0001 C CNN "MFR"
@@
 AR Path="/59ED3D94/59ED1B39" Ref="C11"  Part="1"
 AR Path="/59ED3DAD/59ED1B39" Ref="C18"  Part="1"
-F 0 "C11" H 6625 4150 50  0000 L CNN
+F 0 "C32" H 6625 4150 50  0000 L CNN
 F 1 "10uF" H 6625 3950 50  0000 L CNN
-F 2 "Capacitor_Tantalum_SMD:CP_EIA-3216-18_Kemet-A_Pad1.58x1.35mm_HandSolder" H 6600 4050 50  0001 C CNN
+F 2 "Capacitor_Tantalum_SMD:CP_EIA-2012-12_Kemet-R" H 6600 4050 50  0001 C CNN
 F 3 "" H 6600 4050 50  0001 C CNN
 F 4 "F930J106KAA" H 6600 4050 60  0001 C CNN "MPN"
@@
 AR Path="/59ED3D94/59ED27B9" Ref="L1"  Part="1"
 AR Path="/59ED3DAD/59ED27B9" Ref="L2"  Part="1"
-F 0 "L1" V 6150 2300 50  0000 L CNN
+F 0 "L4" V 6150 2300 50  0000 L CNN
 F 1 "MMZ2012Y152B " V 6075 2300 50  0000 L CNN
 F 2 "Inductor_SMD:L_0805_2012Metric_Pad1.15x1.40mm_HandSolder" V 5930 2350 50  0001 C CNN
@@
 AR Path="/59ED3D94/5A493E0D" Ref="C5"  Part="1"
 AR Path="/59ED3DAD/5A493E0D" Ref="C12"  Part="1"
-F 0 "C5" H 4325 2000 50  0000 L CNN
+F 0 "C26" H 4325 2000 50  0000 L CNN
 F 1 "0.1uF" H 4400 1900 50  0000 L CNN
-F 2 "Capacitor_SMD:C_0805_2012Metric_Pad1.15x1.40mm_HandSolder" H 4338 1750 50  0001 C CNN
+F 2 "Capacitor_SMD:C_0402_1005Metric" H 4338 1750 50  0001 C CNN
 F 3 "" H 4300 1900 50  0001 C CNN
 F 4 "GRM31C5C1E104JA01L " H 4300 1900 60  0001 C CNN "Part"
@@
 AR Path="/59ED3D94/5A493E6F" Ref="C6"  Part="1"
 AR Path="/59ED3DAD/5A493E6F" Ref="C13"  Part="1"
-F 0 "C6" H 3875 2700 50  0000 L CNN
+F 0 "C27" H 3875 2700 50  0000 L CNN
 F 1 "0.1uF" H 3950 2600 50  0000 L CNN
-F 2 "Capacitor_SMD:C_0805_2012Metric_Pad1.15x1.40mm_HandSolder" H 3888 2450 50  0001 C CNN
+F 2 "Capacitor_SMD:C_0402_1005Metric" H 3888 2450 50  0001 C CNN
 F 3 "" H 3850 2600 50  0001 C CNN
 F 4 "GRM31C5C1E104JA01L " H 3850 2600 60  0001 C CNN "Part"
@@
 	3800 3450 4050 3450
 $Comp
-L Slush01:AD8276ARMZ IC11
+L Slush02:AD8276ARMZ IC11
 U 1 1 5D4297EE
 P 2600 1650
@@
 AR Path="/59ED3D94/5D4297EE" Ref="IC2"  Part="1"
 AR Path="/59ED3DAD/5D4297EE" Ref="IC5"  Part="1"
-F 0 "IC2" H 3150 1917 50  0000 C CNN
+F 0 "IC11" H 3150 1917 50  0000 C CNN
 F 1 "AD8276ARMZ" H 3150 1826 50  0000 C CNN
-F 2 "Slush01:MSOP-8" H 3150 1100 50  0001 C CNN
+F 2 "Slush02:MSOP-8" H 3150 1100 50  0001 C CNN
 F 3 "http://docs-europe.electrocomponents.com/webdocs/10ad/0900766b810adb2e.pdf" H 3150 1000 50  0001 C CNN
 F 4 "Analog Devices AD8276ARMZ, Differential Amplifier 0.55MHz Rail to Rail Output 8-pin MSOP" H 3150 900 50  0001 C CNN "Description"
@@
 $EndComp
 $Comp
-L Slush01:AD8603AUJZ-R2 IC12
+L Slush02:AD8603AUJZ-R2 IC12
 U 1 1 5D429956
 P 2650 2600
@@
 AR Path="/59ED3D94/5D429956" Ref="IC3"  Part="1"
 AR Path="/59ED3DAD/5D429956" Ref="IC6"  Part="1"
-F 0 "IC3" H 3100 2867 50  0000 C CNN
+F 0 "IC12" H 3100 2867 50  0000 C CNN
 F 1 "AD8603AUJZ-R2" H 3100 2776 50  0000 C CNN
-F 2 "Slush01:TSOT-23-5" H 3100 2150 50  0001 C CNN
+F 2 "Slush02:TSOT-23-5" H 3100 2150 50  0001 C CNN
 F 3 "http://componentsearchengine.com/Datasheets/3/AD8603AUJZ-R2.pdf" H 3100 2050 50  0001 C CNN
 F 4 "AD8603AUJZ-R2, Operational Amplifier 0.4MHz CMOS, Rail-Rail, 3 V, 5-Pin TSOT" H 3100 1950 50  0001 C CNN "Description"
@@
 $EndComp
 $Comp
-L Slush01:AD8237ARMZ IC13
+L Slush02:AD8237ARMZ IC13
 U 1 1 5D429A53
 P 5400 3400
@@
 AR Path="/59ED3D94/5D429A53" Ref="IC4"  Part="1"
 AR Path="/59ED3DAD/5D429A53" Ref="IC7"  Part="1"
-F 0 "IC4" H 5900 3667 50  0000 C CNN
+F 0 "IC13" H 5900 3667 50  0000 C CNN
 F 1 "AD8237ARMZ" H 5900 3576 50  0000 C CNN
-F 2 "Slush01:MSOP-8" H 5900 2850 50  0001 C CNN
+F 2 "Slush02:MSOP-8" H 5900 2850 50  0001 C CNN
 F 3 "http://www.analog.com/media/en/technical-documentation/data-sheets/AD8237.pdf" H 5900 2750 50  0001 C CNN
 F 4 "Instrumentation Amp Micropower RRIO MSOP Analog Devices AD8237ARMZ Instrumentation Amplifier, 75V Offset 6MHz GBW, CMMR 106dB, 1.8  5.5 V, 8-Pin MSOP" H 5900 2650 50  0001 C CNN "Description"
