File: KiCAD/Igloo10/Igloo10.kicad_pcb (KiCad board)
At the start: 2 copper layers, 40 x 40 mm, 4 parts, among them J1 LSHM-110-01-L-RH-A-S-TR, J2 LSHM-110-01-L-RH-A-S-TR, U1 TEST_PAD, U2 TEST_PAD

Commit message: finished Igloo10
Parts:
- J1, J2: value LSHM-110-01-L-RH-A-S-TR -> LSHM-120-01-L-RH-A-S-TR
Connections:
- J1 pad 10: GND -> Net-(J1-Pad10)
- J1 pad 12: Net-(J1-Pad12) -> GND
- J1 pad 14: GND -> Net-(J1-Pad14)
- J1 pad 16: Net-(J1-Pad16) -> GND
- J1 pad 18: GND -> Net-(J1-Pad18)
- J1 pad 2: GND -> Net-(J1-Pad2)
- J1 pad 20: Net-(J1-Pad20) -> GND
- J1 pad 22: GND -> Net-(J1-Pad22)
- J1 pad 24: Net-(J1-Pad24) -> GND
- J1 pad 26: GND -> Net-(J1-Pad26)
- J1 pad 28: Net-(J1-Pad28) -> GND
- J1 pad 30: GND -> Net-(J1-Pad30)
- J1 pad 32: Net-(J1-Pad32) -> GND
- J1 pad 34: GND -> Net-(J1-Pad34)
- J1 pad 36: Net-(J1-Pad36) -> GND
- J1 pad 38: GND -> Net-(J1-Pad38)
- J1 pad 4: Net-(J1-Pad4) -> GND
- J1 pad 40: Net-(J1-Pad40) -> GND
- J1 pad 6: GND -> Net-(J1-Pad6)
- J1 pad 8: Net-(J1-Pad8) -> GND
- J2 pad 10: GND -> Net-(J2-Pad10)
- J2 pad 12: Net-(J2-Pad12) -> GND
- J2 pad 14: GND -> Net-(J2-Pad14)
- J2 pad 16: Net-(J2-Pad16) -> GND
- J2 pad 18: GND -> Net-(J2-Pad18)
- J2 pad 2: GND -> Net-(J2-Pad2)
- J2 pad 20: Net-(J2-Pad20) -> GND
- J2 pad 22: GND -> Net-(J2-Pad22)
- J2 pad 24: Net-(J2-Pad24) -> GND
- J2 pad 26: GND -> Net-(J2-Pad26)
- J2 pad 28: Net-(J2-Pad28) -> GND
- J2 pad 30: GND -> Net-(J2-Pad30)
- J2 pad 32: Net-(J2-Pad32) -> GND
- J2 pad 34: GND -> Net-(J2-Pad34)
- J2 pad 36: Net-(J2-Pad36) -> GND
- J2 pad 38: GND -> Net-(J2-Pad38)
- J2 pad 4: Net-(J2-Pad4) -> GND
- J2 pad 40: Net-(J2-Pad40) -> GND
- J2 pad 6: GND -> Net-(J2-Pad6)
- J2 pad 8: Net-(J2-Pad8) -> GND
- U1 pad 1: Net-(J1-Pad40) -> Net-(J1-Pad38)
- U1 pad 10: Net-(J1-Pad4) -> Net-(J1-Pad2)
- U1 pad 2: Net-(J1-Pad36) -> Net-(J1-Pad34)
- U1 pad 3: Net-(J1-Pad32) -> Net-(J1-Pad30)
- U1 pad 4: Net-(J1-Pad28) -> Net-(J1-Pad26)
- U1 pad 5: Net-(J1-Pad24) -> Net-(J1-Pad22)
- U1 pad 6: Net-(J1-Pad20) -> Net-(J1-Pad18)
- U1 pad 7: Net-(J1-Pad16) -> Net-(J1-Pad14)
- U1 pad 8: Net-(J1-Pad12) -> Net-(J1-Pad10)
- U1 pad 9: Net-(J1-Pad8) -> Net-(J1-Pad6)
- U2 pad 1: Net-(J2-Pad40) -> Net-(J2-Pad38)
- U2 pad 10: Net-(J2-Pad4) -> Net-(J2-Pad2)
- U2 pad 2: Net-(J2-Pad36) -> Net-(J2-Pad34)
- U2 pad 3: Net-(J2-Pad32) -> Net-(J2-Pad30)
- U2 pad 4: Net-(J2-Pad28) -> Net-(J2-Pad26)
- U2 pad 5: Net-(J2-Pad24) -> Net-(J2-Pad22)
- U2 pad 6: Net-(J2-Pad20) -> Net-(J2-Pad18)
- U2 pad 7: Net-(J2-Pad16) -> Net-(J2-Pad14)
- U2 pad 8: Net-(J2-Pad12) -> Net-(J2-Pad10)
- U2 pad 9: Net-(J2-Pad8) -> Net-(J2-Pad6)
Routing:
- net GND: track 0.00 -> 17.1 mm
- net Net-(J2-Pad38): track 0.00 -> 7.08 mm, vias 0 -> 1
- net Net-(J1-Pad4): track 7.05 -> 0.00 mm, vias 1 -> 0
- net Net-(J1-Pad38): track 0.00 -> 7.05 mm, vias 0 -> 1
- net Net-(J2-Pad34): track 0.00 -> 7.02 mm, vias 0 -> 1
- net Net-(J1-Pad8): track 6.99 -> 0.00 mm, vias 1 -> 0
- net Net-(J1-Pad34): track 0.00 -> 6.99 mm, vias 0 -> 1
- net Net-(J2-Pad30): track 0.00 -> 6.96 mm, vias 0 -> 1
- net Net-(J1-Pad30): track 0.00 -> 6.93 mm, vias 0 -> 1
- net Net-(J1-Pad12): track 6.93 -> 0.00 mm, vias 1 -> 0
- net Net-(J2-Pad26): track 0.00 -> 6.90 mm, vias 0 -> 1
- net Net-(J2-Pad2): track 0.00 -> 6.87 mm, vias 0 -> 1
- net Net-(J1-Pad26): track 0.00 -> 6.87 mm, vias 0 -> 1
- net Net-(J1-Pad16): track 6.87 -> 0.00 mm, vias 1 -> 0
- net Net-(J2-Pad22): track 0.00 -> 6.84 mm, vias 0 -> 1
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Other:
- rule trace_min: 0.2 -> 0.1524
