File: KiCAD/Igloo10/Igloo10.sch (KiCad schematic (older format))
At the start: 4 parts, among them J1 LSHM-110-01-L-RH-A-S-TR, J2 LSHM-110-01-L-RH-A-S-TR, U1 TEST_PAD, U2 TEST_PAD

Commit message: finished Igloo10
Parts:
- removed J1, J2: LSHM-110-01-L-RH-A-S-TR, Igloo10:LSHM-110-01-L-RH-A-S-TR, symbol Igloo10:LSHM-110-01-L-RH-A-S-TR
- added J1, J2: LSHM-120-01-L-RH-A-S-TR, Igloo10:LSHM-120-01-L-RH-A-S-TR, symbol Igloo10:LSHM-120-01-L-RH-A-S-TR
Other:
- moved on the sheet: U1
