File: KiCAD/Straightener01/Straightener01.sch (KiCad schematic (older format))
At the start: 13 parts, among them IC1 LT3045EDD, J1 C112640, J2 C112640

Commit message: finished up Straightener01
Parts:
- C1: footprint Capacitor_SMD:CP_Elec_6.3x5.4 -> Capacitor_SMD:CP_Elec_5x5.3
Changed lines of the file:
@@
 F 0 "C1" H 5300 2700 50  0000 R CNN
 F 1 "22uF" H 5300 2600 50  0000 R CNN
-F 2 "Capacitor_SMD:CP_Elec_6.3x5.4" H 5400 2650 50  0001 C CNN
+F 2 "Capacitor_SMD:CP_Elec_5x5.3" H 5400 2650 50  0001 C CNN
 F 3 "~" H 5400 2650 50  0001 C CNN
 	1    5400 2650
