File: KiCAD/Gateway04/Gateway04.sch (KiCad schematic (older format))
At the start: 8 parts, among them U1 LSHM-120-02.5-L-DV-A-S-TR, U2 LSHM-120-02.5-L-DV-A-S-TR, U3 LSHM-120-02.5-L-DV-A-S-TR, U4 LSHM-120-02.5-L-DV-A-S-TR, U5 LSHM-120-02.5-L-DV-A-S-TR, U6 LSHM-120-02.5-L-DV-A-S-TR, U7 LSHM-120-02.5-L-DV-A-S-TR, U8 LSHM-120-02.5-L-DV-A-S-TR

Commit message: finished Gateway04
Parts:
- U1, U2, U3, U4, U5, U6, U7, U8: footprint Gateway03:LSHM-120-02.5-L-DV-A-S-TR -> Gateway04:LSHM-120-02.5-L-DV-A-S-TR; symbol Gateway03:LSHM-120-02.5-L-DV-A-S-TR -> Gateway04:LSHM-120-02.5-L-DV-A-S-TR
Changed lines of the file:
@@
 Connection ~ 7400 3350
 $Comp
-L Gateway03:LSHM-120-02.5-L-DV-A-S-TR U2
+L Gateway04:LSHM-120-02.5-L-DV-A-S-TR U2
 U 1 1 5DD1749D
 P 2000 1550
 F 0 "U2" H 2000 2265 50  0000 C CNN
 F 1 "LSHM-120-02.5-L-DV-A-S-TR" H 2000 2174 50  0000 C CNN
-F 2 "Gateway03:LSHM-120-02.5-L-DV-A-S-TR" H 2000 2250 50  0001 C CNN
+F 2 "Gateway04:LSHM-120-02.5-L-DV-A-S-TR" H 2000 2250 50  0001 C CNN
 F 3 "" H 2000 2250 50  0001 C CNN
 	1    2000 1550
@@
 $EndComp
 $Comp
-L Gateway03:LSHM-120-02.5-L-DV-A-S-TR U4
+L Gateway04:LSHM-120-02.5-L-DV-A-S-TR U4
 U 1 1 5DD183C7
 P 4150 1550
 F 0 "U4" H 4150 2265 50  0000 C CNN
 F 1 "LSHM-120-02.5-L-DV-A-S-TR" H 4150 2174 50  0000 C CNN
-F 2 "Gateway03:LSHM-120-02.5-L-DV-A-S-TR" H 4150 2250 50  0001 C CNN
+F 2 "Gateway04:LSHM-120-02.5-L-DV-A-S-TR" H 4150 2250 50  0001 C CNN
 F 3 "" H 4150 2250 50  0001 C CNN
 	1    4150 1550
@@
 $EndComp
 $Comp
-L Gateway03:LSHM-120-02.5-L-DV-A-S-TR U6
+L Gateway04:LSHM-120-02.5-L-DV-A-S-TR U6
 U 1 1 5DD19DEE
 P 6300 1550
 F 0 "U6" H 6300 2265 50  0000 C CNN
 F 1 "LSHM-120-02.5-L-DV-A-S-TR" H 6300 2174 50  0000 C CNN
-F 2 "Gateway03:LSHM-120-02.5-L-DV-A-S-TR" H 6300 2250 50  0001 C CNN
+F 2 "Gateway04:LSHM-120-02.5-L-DV-A-S-TR" H 6300 2250 50  0001 C CNN
 F 3 "" H 6300 2250 50  0001 C CNN
 	1    6300 1550
@@
 $EndComp
 $Comp
-L Gateway03:LSHM-120-02.5-L-DV-A-S-TR U8
+L Gateway04:LSHM-120-02.5-L-DV-A-S-TR U8
 U 1 1 5DD1B1EE
 P 8450 1550
 F 0 "U8" H 8450 2265 50  0000 C CNN
 F 1 "LSHM-120-02.5-L-DV-A-S-TR" H 8450 2174 50  0000 C CNN
-F 2 "Gateway03:LSHM-120-02.5-L-DV-A-S-TR" H 8450 2250 50  0001 C CNN
+F 2 "Gateway04:LSHM-120-02.5-L-DV-A-S-TR" H 8450 2250 50  0001 C CNN
 F 3 "" H 8450 2250 50  0001 C CNN
 	1    8450 1550
@@
 $EndComp
 $Comp
-L Gateway03:LSHM-120-02.5-L-DV-A-S-TR U7
+L Gateway04:LSHM-120-02.5-L-DV-A-S-TR U7
 U 1 1 5DD4BF27
 P 7750 1650
 F 0 "U7" H 7750 2365 50  0000 C CNN
 F 1 "LSHM-120-02.5-L-DV-A-S-TR" H 7750 2274 50  0000 C CNN
-F 2 "Gateway03:LSHM-120-02.5-L-DV-A-S-TR" H 7750 2350 50  0001 C CNN
+F 2 "Gateway04:LSHM-120-02.5-L-DV-A-S-TR" H 7750 2350 50  0001 C CNN
 F 3 "" H 7750 2350 50  0001 C CNN
 	1    7750 1650
@@
 $EndComp
 $Comp
-L Gateway03:LSHM-120-02.5-L-DV-A-S-TR U5
+L Gateway04:LSHM-120-02.5-L-DV-A-S-TR U5
 U 1 1 5DD790BA
 P 5600 1650
 F 0 "U5" H 5600 2365 50  0000 C CNN
 F 1 "LSHM-120-02.5-L-DV-A-S-TR" H 5600 2274 50  0000 C CNN
-F 2 "Gateway03:LSHM-120-02.5-L-DV-A-S-TR" H 5600 2350 50  0001 C CNN
+F 2 "Gateway04:LSHM-120-02.5-L-DV-A-S-TR" H 5600 2350 50  0001 C CNN
 F 3 "" H 5600 2350 50  0001 C CNN
 	1    5600 1650
@@
 $EndComp
 $Comp
-L Gateway03:LSHM-120-02.5-L-DV-A-S-TR U1
+L Gateway04:LSHM-120-02.5-L-DV-A-S-TR U1
 U 1 1 5DDD27B8
 P 1300 1650
 F 0 "U1" H 1300 2365 50  0000 C CNN
 F 1 "LSHM-120-02.5-L-DV-A-S-TR" H 1300 2274 50  0000 C CNN
-F 2 "Gateway03:LSHM-120-02.5-L-DV-A-S-TR" H 1300 2350 50  0001 C CNN
+F 2 "Gateway04:LSHM-120-02.5-L-DV-A-S-TR" H 1300 2350 50  0001 C CNN
 F 3 "" H 1300 2350 50  0001 C CNN
 	1    1300 1650
@@
 $EndComp
 $Comp
-L Gateway03:LSHM-120-02.5-L-DV-A-S-TR U3
+L Gateway04:LSHM-120-02.5-L-DV-A-S-TR U3
 U 1 1 5DE0B6F8
 P 3450 1650
 F 0 "U3" H 3450 2365 50  0000 C CNN
 F 1 "LSHM-120-02.5-L-DV-A-S-TR" H 3450 2274 50  0000 C CNN
-F 2 "Gateway03:LSHM-120-02.5-L-DV-A-S-TR" H 3450 2350 50  0001 C CNN
+F 2 "Gateway04:LSHM-120-02.5-L-DV-A-S-TR" H 3450 2350 50  0001 C CNN
 F 3 "" H 3450 2350 50  0001 C CNN
 	1    3450 1650
